File: SignControlBoard/LED sign board 3.sch (EAGLE design)
At the start: 45 parts, among them IC1 MSGEQ7DIL, U1 ATMEGA328P, U2 M5205 5v, Y1 16MHz

Commit message: Updated LED Boards
Parts:
- removed C11: 0.01uf, eagle-ltspice:CC0201
- removed C12, C13: 0.1uf, eagle-ltspice:CC0201
- removed C14: 33pf, eagle-ltspice:CC0201
- added C10: 33pf, capacitor-wima:C2,5-3
- added C7: 10uF, SparkFun-Passives:CAP_POL1206
- added C8, C9: 0.1uf, capacitor-wima:C2,5-3
- C4: value 10uF -> 0.01uf; device SparkFun-Passives:CAP_POL1206 -> capacitor-wima:C2,5-3
Connections:
- net GND: now also C10.2, C7.-, C8.2, C9.2; no longer C12.2, C13.2, C14.2, C4.-
- net N$10: now also C4.2; no longer C11.2
- net N$11: now also C9.1; no longer C13.1
- net N$12: now also C10.1; no longer C14.1
- net N$9: now also C4.1; no longer C11.1
- net VCC: now also C8.1; no longer C12.1
- net VIN: now also C7.+; no longer C4.+
Changed lines of the file:
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@@
 <part name="U2" library="SparkFun-PowerIC" deviceset="MIC5205" device="5V" value="M5205 5v"/>
 <part name="GND6" library="SparkFun-Aesthetics" deviceset="GND" device=""/>
-<part name="C4" library="SparkFun-Passives" deviceset="CAP_POL" device="1206" value="10uF"/>
 <part name="GND7" library="SparkFun-Aesthetics" deviceset="GND" device=""/>
 <part name="C5" library="SparkFun-Passives" deviceset="CAP_POL" device="1206" value="10uF"/>
@@
 <part name="IC1" library="SparkFun-AnalogIC" deviceset="MSGEQ7" device="DIL"/>
 <part name="SL1" library="con-amp-quick" deviceset="M03" device=""/>
-<part name="C11" library="eagle-ltspice" deviceset="C" device="C0201" value="0.01uf"/>
-<part name="C12" library="eagle-ltspice" deviceset="C" device="C0201" value="0.1uf"/>
-<part name="C13" library="eagle-ltspice" deviceset="C" device="C0201" value="0.1uf"/>
-<part name="C14" library="eagle-ltspice" deviceset="C" device="C0201" value="33pf"/>
 <part name="SL2" library="con-amp-quick" deviceset="M04" device=""/>
 <part name="SL3" library="con-amp-quick" deviceset="M04" device=""/>
@@
 <part name="JP2" library="SparkFun-Connectors" deviceset="POWER_JACK" device="PTH"/>
 <part name="SL10" library="con-amp-quick" deviceset="M02" device=""/>
+<part name="C7" library="SparkFun-Passives" deviceset="CAP_POL" device="1206" value="10uF"/>
+<part name="C4" library="capacitor-wima" deviceset="C" device="2,5-3" value="0.01uf"/>
+<part name="C8" library="capacitor-wima" deviceset="C" device="2,5-3" value="0.1uf"/>
+<part name="C9" library="capacitor-wima" deviceset="C" device="2,5-3" value="0.1uf"/>
+<part name="C10" library="capacitor-wima" deviceset="C" device="2,5-3" value="33pf"/>
 </parts>
 <sheets>
@@
 <instance part="U2" gate="G$1" x="-33.02" y="73.66"/>
 <instance part="GND6" gate="1" x="-48.26" y="58.42"/>
-<instance part="C4" gate="G$1" x="-66.04" y="71.12"/>
 <instance part="GND7" gate="1" x="-66.04" y="58.42"/>
 <instance part="C5" gate="G$1" x="-7.62" y="73.66"/>
@@
 <instance part="IC1" gate="G$1" x="236.22" y="63.5"/>
 <instance part="SL1" gate="G$1" x="190.5" y="86.36"/>
-<instance part="C11" gate="G$1" x="198.12" y="76.2"/>
-<instance part="C12" gate="G$1" x="215.9" y="53.34"/>
-<instance part="C13" gate="G$1" x="266.7" y="53.34"/>
-<instance part="C14" gate="G$1" x="276.86" y="53.34"/>
 <instance part="SL2" gate="G$1" x="160.02" y="-58.42" rot="R90"/>
 <instance part="SL3" gate="G$1" x="182.88" y="-58.42" rot="R90"/>
@@
 <instance part="JP2" gate="G$1" x="-35.56" y="-27.94" rot="R180"/>
 <instance part="SL10" gate="G$1" x="-50.8" y="-45.72" rot="R90"/>
+<instance part="C7" gate="G$1" x="-66.04" y="71.12"/>
+<instance part="C4" gate="G$1" x="198.12" y="76.2"/>
+<instance part="C8" gate="G$1" x="215.9" y="53.34"/>
+<instance part="C9" gate="G$1" x="266.7" y="53.34"/>
+<instance part="C10" gate="G$1" x="276.86" y="53.34"/>
 </instances>
 <busses>
@@
 </segment>
 <segment>
-<pinref part="C4" gate="G$1" pin="-"/>
 <wire x1="-66.04" y1="66.04" x2="-66.04" y2="60.96" width="0.1524" layer="91"/>
 <pinref part="GND7" gate="1" pin="GND"/>
+<pinref part="C7" gate="G$1" pin="-"/>
 </segment>
 <segment>
@@
 <junction x="276.86" y="40.64"/>
 <label x="302.26" y="40.64" size="1.778" layer="95"/>
-<pinref part="C12" gate="G$1" pin="2"/>
-<pinref part="C13" gate="G$1" pin="2"/>
-<pinref part="C14" gate="G$1" pin="2"/>
 <pinref part="IC1" gate="G$1" pin="CG"/>
 <wire x1="251.46" y1="63.5" x2="256.54" y2="63.5" width="0.1524" layer="91"/>
+<pinref part="C8" gate="G$1" pin="2"/>
+<pinref part="C9" gate="G$1" pin="2"/>
+<pinref part="C10" gate="G$1" pin="2"/>
 </segment>
 <segment>
@@
 <wire x1="218.44" y1="68.58" x2="215.9" y2="68.58" width="0.1524" layer="91"/>
 <junction x="215.9" y="68.58"/>
-<pinref part="C12" gate="G$1" pin="1"/>
 <pinref part="R9" gate="G$1" pin="2"/>
+<pinref part="C8" gate="G$1" pin="1"/>
 </segment>
 <segment>
@@
 <junction x="-53.34" y="78.74"/>
 <label x="-73.66" y="78.74" size="1.778" layer="95" rot="R180" xref="yes"/>
-<pinref part="C4" gate="G$1" pin="+"/>
 <wire x1="-66.04" y1="73.66" x2="-66.04" y2="78.74" width="0.1524" layer="91"/>
 <junction x="-66.04" y="78.74"/>
+<pinref part="C7" gate="G$1" pin="+"/>
 </segment>
 <segment>
@@
 <pinref part="SL1" gate="G$1" pin="1"/>
 <wire x1="198.12" y1="83.82" x2="198.12" y2="78.74" width="0.1524" layer="91"/>
-<pinref part="C11" gate="G$1" pin="1"/>
+<pinref part="C4" gate="G$1" pin="1"/>
 </segment>
 </net>
@@
 <pinref part="IC1" gate="G$1" pin="AUDIO_IN"/>
 <wire x1="198.12" y1="66.04" x2="218.44" y2="66.04" width="0.1524" layer="91"/>
-<pinref part="C11" gate="G$1" pin="2"/>
+<pinref part="C4" gate="G$1" pin="2"/>
 </segment>
 </net>
@@
 <wire x1="251.46" y1="60.96" x2="266.7" y2="60.96" width="0.1524" layer="91"/>
 <wire x1="266.7" y1="60.96" x2="266.7" y2="55.88" width="0.1524" layer="91"/>
-<pinref part="C13" gate="G$1" pin="1"/>
+<pinref part="C9" gate="G$1" pin="1"/>
 </segment>
 </net>
@@
 <wire x1="276.86" y1="71.12" x2="276.86" y2="66.04" width="0.1524" layer="91"/>
 <junction x="276.86" y="66.04"/>
-<pinref part="C14" gate="G$1" pin="1"/>
 <pinref part="R9" gate="G$1" pin="1"/>
-</segment>
-</net>
+<pinref part="C10" gate="G$1" pin="1"/>
+</segment>
+</net>
